File: impregnator-adaptor-board.kicad_pcb (KiCad board)
At the start: 2 copper layers, 116 x 174.9 mm, 20 parts, among them J1 1932588, J10 1935336, J11 Conn_01x16_Socket, J12 Conn_01x16_Socket, J13 Conn_01x24_Socket, J14 Conn_01x24_Socket, J15 1935336, J16 1935336, J2 Conn_01x16_Socket, J3 Conn_01x16_Socket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

Commit message: project native components
Parts:
- J1: footprint 1932588:PHOENIX_1932588 -> impregnator-adaptor-board:PHOENIX_1932588
- J10, J15, J16, J8, J9: footprint 1935336:PHOENIX_1935336 -> impregnator-adaptor-board:PHOENIX_1935336
Changed lines of the file:
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@@
 	)
 	(setup
+		(stackup
+			(layer "F.SilkS"
+				(type "Top Silk Screen")
+			)
+			(layer "F.Paste"
+				(type "Top Solder Paste")
+			)
+			(layer "F.Mask"
+				(type "Top Solder Mask")
+				(thickness 0.01)
+			)
+			(layer "F.Cu"
+				(type "copper")
+				(thickness 0.035)
+			)
+			(layer "dielectric 1"
+				(type "core")
+				(thickness 1.51)
+				(material "FR4")
+				(epsilon_r 4.5)
+				(loss_tangent 0.02)
+			)
+			(layer "B.Cu"
+				(type "copper")
+				(thickness 0.035)
+			)
+			(layer "B.Mask"
+				(type "Bottom Solder Mask")
+				(thickness 0.01)
+			)
+			(layer "B.Paste"
+				(type "Bottom Solder Paste")
+			)
+			(layer "B.SilkS"
+				(type "Bottom Silk Screen")
+			)
+			(copper_finish "None")
+			(dielectric_constraints no)
+		)
 		(pad_to_mask_clearance 0)
 		(allow_soldermask_bridges_in_footprints no)
@@
 	(net 24 "/E2+")
 	(net 25 "/E1-")
-	(footprint "1935336:PHOENIX_1935336"
+	(footprint "impregnator-adaptor-board:PHOENIX_1935336"
 		(layer "F.Cu")
 		(at 109.5125 118.06)
@@
 		(embedded_fonts no)
 	)
-	(footprint "1935336:PHOENIX_1935336"
+	(footprint "impregnator-adaptor-board:PHOENIX_1935336"
 		(layer "F.Cu")
 		(at 109.5125 188.67)
@@
 		(embedded_fonts no)
 	)
-	(footprint "1935336:PHOENIX_1935336"
+	(footprint "impregnator-adaptor-board:PHOENIX_1935336"
 		(layer "F.Cu")
 		(at 44.0875 16.44 180)
 		(property "Reference" "J8"
-			(at 3.175 -12.385 0)
+			(at 3.175 -12.385 180)
 			(layer "F.SilkS")
 			(effects
@@
 		)
 		(property "Value" "1935336"
-			(at 9.525 1.115 0)
+			(at 9.525 1.115 180)
 			(layer "F.Fab")
 			(effects
@@
 		)
 		(property "Datasheet" ""
-			(at 0 0 0)
+			(at 0 0 180)
 			(layer "F.Fab")
 			(hide yes)
@@
 		)
 		(property "Description" ""
-			(at 0 0 0)
+			(at 0 0 180)
 			(layer "F.Fab")
 			(hide yes)
@@
 		(embedded_fonts no)
 	)
-	(footprint "1935336:PHOENIX_1935336"
+	(footprint "impregnator-adaptor-board:PHOENIX_1935336"
 		(layer "F.Cu")
 		(at 126.9 41.4775 90)
@@
 		(embedded_fonts no)
 	)
-	(footprint "1932588:PHOENIX_1932588"
+	(footprint "impregnator-adaptor-board:PHOENIX_1932588"
 		(layer "F.Cu")
 		(at 63.35 113.4125)
@@
 		(embedded_fonts no)
 	)
-	(footprint "1935336:PHOENIX_1935336"
+	(footprint "impregnator-adaptor-board:PHOENIX_1935336"
 		(layer "F.Cu")
 		(at 44.0875 87.05 180)
 		(property "Reference" "J9"
-			(at 3.175 -12.385 0)
+			(at 3.175 -12.385 180)
 			(layer "F.SilkS")
 			(effects
@@
 		)
 		(property "Value" "1935336"
-			(at 9.525 1.115 0)
+			(at 9.525 1.115 180)
 			(layer "F.Fab")
 			(effects
@@
 		)
 		(property "Datasheet" ""
-			(at 0 0 0)
+			(at 0 0 180)
 			(layer "F.Fab")
 			(hide yes)
@@
 		)
 		(property "Description" ""
-			(at 0 0 0)
-			(layer "F.Fab")
-			(hide yes)
+			(at 0 0 180)
+			(layer "F.Fab")
+			(hide yes)

Commit message: use smaller central screw connector
Parts:
- J1: value 1932588 -> 1773976; footprint impregnator-adaptor-board:PHOENIX_1932588 -> impregnator-adaptor-board:PHOENIX_1773976
- moved J1 12.4 mm to (68.1, 102.0)
Routing:
- net /VIN: track 212.9 -> 162.5 mm
- net /C1+: track 16.8 -> 17.3 mm
