File: impregnator-adaptor-board.kicad_pcb (KiCad board)
At the start: 2 copper layers, 116 x 174.9 mm, 20 parts, among them J1 1773976, J10 1935336, J11 Conn_01x16_Socket, J12 Conn_01x16_Socket, J13 Conn_01x24_Socket, J14 Conn_01x24_Socket, J15 1935336, J16 1935336, J2 Conn_01x16_Socket, J3 Conn_01x16_Socket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

Commit message: put all slots on the same side and add silkscreen
Parts:
- added H5: MountingHole_Pad, MountingHole:MountingHole_3.2mm_M3_DIN965_Pad, F.Cu at (357.5, 121.5)
- moved H4 279.9 mm to (357.5, 87.2), turned to 180 degrees
- moved J12 277.1 mm to (344.7, 95.9), turned to 180 degrees
- moved H2 227.4 mm to (357.5, 54.8), turned to 180 degrees
- moved J14 207.6 mm to (309.1, 95.9), turned to 180 degrees
- moved J11 183.5 mm to (284.7, 95.9), turned to 180 degrees
- moved J16 178.1 mm to (295.0, 100.4), turned to -90 degrees
- moved J13 161.6 mm to (249.1, 95.9), turned to 180 degrees
- moved J15 153.4 mm to (235.0, 100.4), turned to -90 degrees
- moved J1 142.0 mm to (208.7, 81.6), turned to 90 degrees
- moved H1 134.8 mm to (58.8, 54.8), turned to 180 degrees
- moved J3 124.9 mm to (164.7, 95.9), turned to 180 degrees
- moved J4 123.9 mm to (224.7, 95.9), turned to 180 degrees
- moved J8 84.6 mm to (55.0, 100.4), turned to -90 degrees
- moved J5 84.0 mm to (189.1, 95.9), turned to 180 degrees
- moved J7 81.3 mm to (129.1, 95.9), turned to 180 degrees
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Routing:
- net /VIN: track 162.5 -> 0.00 mm
- net /A1-: track 17.5 -> 12.4 mm
- net /E1-: track 17.3 -> 12.4 mm
- net /B1+: track 17.4 -> 12.5 mm
- net /A2+: track 17.1 -> 12.2 mm
- net /A1+: track 17.4 -> 12.5 mm
- net /B1-: track 17.2 -> 12.4 mm
- net /E1+: track 17.3 -> 12.5 mm
- net /B2+: track 17.0 -> 12.2 mm
- net /C1+: track 17.3 -> 12.5 mm
- net /D1+: track 17.2 -> 12.5 mm
- net /B2-: track 16.9 -> 12.2 mm
- net /C1-: track 17.1 -> 12.4 mm
- net /C2-: track 16.8 -> 12.2 mm
- net /C2+: track 16.8 -> 12.2 mm
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Other:
- board size 116 x 174.9 mm -> 306.9 x 75 mm
- board text added: "A1+"
- board text added: "A1-"
- board text added: "A2+"
- board text added: "A2-"
- board text added: "B1+"
- board text added: "B1-"
- board text added: "B2+"
- board text added: "B2-"
- board text added: "C1+"
- board text added: "C1-"
- board text added: "C2+"
- board text added: "C2-"
- board text added: "D1+"
- board text added: "D1-"
- board text added: "D2+"
- board text added: "D2-"
- board text added: "E1+"
- board text added: "E1-"
- board text added: "E2+"
- board text added: "E2-"
- board text added: "GND"
- board text added: "VIN"
